File: BQ2xxxx/BQ2xxxx.kicad_pcb (KiCad board)
At the start: 2 copper layers, 8 parts, among them J1 1054500101, J2 1054500101, U1 BQ25895MRTWT, U2 BQ24296MRGER

Commit message: MAIN: 25.06.2025
Parts:
- removed TP1: +5V, TestPoint:TestPoint_Pad_D3.0mm
- removed TP2: GND, TestPoint:TestPoint_Pad_D3.0mm
- added C1: 0.1u, Capacitor_SMD:C_0603_1608Metric, F.Cu at (93.7, 59.9)
- added C3: 10u, Capacitor_SMD:C_0603_1608Metric, F.Cu at (60.4, 83.5)
- added C4: 33u, Capacitor_SMD:C_0603_1608Metric, F.Cu at (62.2, 81.7)
- added Cbst1: 100n, Capacitor_SMD:C_0603_1608Metric, F.Cu at (89.7, 31.0)
- added Ccomp1: 39n, Capacitor_SMD:C_0603_1608Metric, F.Cu at (89.7, 33.5)
- added Ccomp2: 82p, Capacitor_SMD:C_0603_1608Metric, F.Cu at (89.7, 36.0)
- added Cin1: 10u, Capacitor_SMD:C_0603_1608Metric, F.Cu at (89.7, 38.5)
- added Cinx1: 100n, Capacitor_SMD:C_0603_1608Metric, F.Cu at (89.7, 41.0)
- added Cout1: 47u, Capacitor_SMD:C_0603_1608Metric, F.Cu at (93.7, 31.0)
- added Cout2: 47u, Capacitor_SMD:C_0603_1608Metric, F.Cu at (93.7, 33.5)
- added Cout3: 47u, Capacitor_SMD:C_0603_1608Metric, F.Cu at (93.7, 36.0)
- added Cvcc1: 2.2u, Capacitor_SMD:C_0603_1608Metric, F.Cu at (93.7, 38.5)
- added HSE1: 8MHz, Crystal:Crystal_SMD_3225-4Pin_3.2x2.5mm, F.Cu at (45.5, 59.2)
- added IC1: STM32F030R8T6, STM32F030R8T6:QFP50P1200X1200X160-64N, F.Cu at (51.3, 75.3)
- added IC2: TPS61288RQQR, SamacSys:TPS61288RQQR, F.Cu at (103.0, 32.7)
- added J4: USB4125-GF-A, SamacSys:USB4125GFA, F.Cu at (25.3, 25.2)
- added L1: 2.2u, Inductor_SMD:L_6.3x6.3_H3, F.Cu at (69.3, 83.5)
- added L2: 1.5u, Inductor_SMD:L_6.3x6.3_H3, F.Cu at (100.0, 41.0)
- added LSE1: 32.768kHz, Crystal:Crystal_SMD_3215-2Pin_3.2x1.5mm, F.Cu at (44.1, 65.8)
- added PS1: TPS25942ARVCT, SamacSys:QFN50P300X400X80-21N, F.Cu at (73.1, 38.0)
- added R1: 5.1k, Resistor_SMD:R_0603_1608Metric, F.Cu at (32.7, 22.4)
- added R2: 5.1k, Resistor_SMD:R_0603_1608Metric, F.Cu at (22.5, 32.6)
- added R3: 10k, Resistor_SMD:R_0603_1608Metric, F.Cu at (107.3, 97.1)
- added R4: 10k, Resistor_SMD:R_0603_1608Metric, F.Cu at (97.1, 107.3)
- added R5: 10k, Resistor_SMD:R_0603_1608Metric, F.Cu at (92.0, 58.1)
- added R6: 10k, Resistor_SMD:R_0603_1608Metric, F.Cu at (90.2, 56.4)
- added R7: 10k, Resistor_SMD:R_0603_1608Metric, F.Cu at (88.4, 54.6)
- added Rcomp1: 35.7k, Resistor_SMD:R_0603_1608Metric, F.Cu at (97.7, 31.0)
- added Rfbb1: 48.7k, Resistor_SMD:R_0603_1608Metric, F.Cu at (97.7, 33.5)
- added Rfbt1: 357k, Resistor_SMD:R_0603_1608Metric, F.Cu at (97.7, 36.0)
- added S1: JS202011JCQN, SamacSys:JS202011JCQN, F.Cu at (26.9, 103.0)
- added U3: CC56-12GWA, Display_7Segment:CC56-12GWA, F.Cu at (22.1, 58.6)
- added U4: CC56-12GWA, Display_7Segment:CC56-12GWA, F.Cu at (58.6, 107.7)
- added U6: AS1115-BSST, Package_SO:QSOP-24_3.9x8.7mm_P0.635mm, F.Cu at (32.8, 96.9)
- added U7: TPS63001, Package_SON:Texas_DRC0010J, F.Cu at (64.4, 86.9)
- J1: value 1054500101 -> USB4125-GF-A; footprint 1054500101:MOLEX_1054500101 -> SamacSys:USB4125GFA
- J2: value 1054500101 -> Conn_01x05; footprint 1054500101:MOLEX_1054500101 -> Connector_PinHeader_2.54mm:PinHeader_1x05_P2.54mm_Vertical
- U1: value BQ25895MRTWT -> MAX17048G_T10; footprint BQ25895MRTWT:QFN50P400X400X80-25N -> MAX17048G_T10:SON50P200X200X80-9N
- moved BT1 145.4 mm to (49.9, 36.4), turned to 45 degrees
- moved J1 95.0 mm to (104.6, 104.5), turned to 45 degrees
- moved U2 80.7 mm to (80.6, 44.9), turned to 45 degrees
- moved U1 67.0 mm to (85.8, 52.9), turned to -135 degrees
- moved BT2 33.9 mm to (92.7, 79.1), turned to -45 degrees
- moved J2 25.9 mm to (96.0, 56.1), turned to -135 degrees
Connections:
- BT1 pad N1: unconnected-(BT1-PadN1) -> GND
- BT1 pad N2: unconnected-(BT1-PadN2) -> GND
- BT1 pad N3: unconnected-(BT1-PadN3) -> GND
- BT2 pad 1_1: unconnected-(BT2-Pad1_1) -> +BATT
- BT2 pad 1_2: unconnected-(BT2-Pad1_2) -> +BATT
- BT2 pad 1_3: unconnected-(BT2-Pad1_3) -> +BATT
- J1 pad A12: unconnected-(J1-GND_A12-PadA12) -> GND
- J1 pad A5: unconnected-(J1-CC1-PadA5) -> Net-(J1-CC1)
- J1 pad A9: unconnected-(J1-VBUS_A9-PadA9) -> +5V
- J1 pad B12: unconnected-(J1-GND_B12-PadB12) -> GND
- J1 pad B5: unconnected-(J1-CC2-PadB5) -> Net-(J1-CC2)
- J1 pad B9: unconnected-(J1-VBUS_B9-PadB9) -> +5V
- U1 pad 1: unconnected-(U1-VBUS-Pad1) -> GND
- U1 pad 2: unconnected-(U1-D+-Pad2) -> +BATT
- U1 pad 3: unconnected-(U1-D–-Pad3) -> +BATT
- U1 pad 4: unconnected-(U1-STAT-Pad4) -> GND
- U1 pad 5: unconnected-(U1-SCL-Pad5) -> /INT
- U1 pad 6: unconnected-(U1-SDA-Pad6) -> GND
- U1 pad 7: unconnected-(U1-INT-Pad7) -> /SCL
- U1 pad 8: unconnected-(U1-OTG-Pad8) -> /SDA
- U1 pad 9: unconnected-(U1-~{CE}-Pad9) -> GND
- U2 pad 2: unconnected-(U2-PSEL-Pad2) -> GND
Other:
- board outline added: 89.8 x 89.8 mm

Commit message: Work in progress: Schematic
Parts:
- removed IC1: STM32F030R8T6, STM32F030R8T6:QFP50P1200X1200X160-64N
- removed LSE1: 32.768kHz, Crystal:Crystal_SMD_3215-2Pin_3.2x1.5mm
- added C10: 10u, Capacitor_SMD:C_0603_1608Metric, F.Cu at (83.4, 32.8)
- added C11: 10n, Capacitor_SMD:C_0402_1005Metric, F.Cu at (85.7, 24.6)
- added C12: 1u, Capacitor_SMD:C_0402_1005Metric, F.Cu at (85.7, 26.6)
- added C13: 1u, Capacitor_SMD:C_0402_1005Metric, F.Cu at (85.7, 28.6)
- added C14: 100n, Capacitor_SMD:C_0402_1005Metric, F.Cu at (85.7, 30.6)
- added C15: 10u, Capacitor_SMD:C_0603_1608Metric, F.Cu at (94.9, 108.9)
- added C2: 22p, Capacitor_SMD:C_0402_1005Metric, F.Cu at (82.9, 22.7)
- added C5: 22p, Capacitor_SMD:C_0402_1005Metric, F.Cu at (82.9, 24.6)
- added C6: 100n, Capacitor_SMD:C_0402_1005Metric, F.Cu at (82.9, 26.6)
- added C7: 100n, Capacitor_SMD:C_0402_1005Metric, F.Cu at (82.9, 28.6)
- added C8: 100n, Capacitor_SMD:C_0402_1005Metric, F.Cu at (82.9, 30.6)
- added C9: 100n, Capacitor_SMD:C_0402_1005Metric, F.Cu at (85.7, 22.7)
- added D1: Blue, LED_SMD:LED_0402_1005Metric, F.Cu at (88.8, 22.7)
- added D2: Blue, LED_SMD:LED_0402_1005Metric, F.Cu at (88.8, 24.7)
- added D3: Green, LED_SMD:LED_0402_1005Metric, F.Cu at (88.8, 26.7)
- added J3: SLW-66527511-SMT-TR, SamacSys:SLW66527511SMTTR, F.Cu at (44.1, 61.7)
- added J5: USB_B_Micro, Connector_USB:USB_Micro-B_Amphenol_10118193-0001LF_Horizontal, F.Cu at (34.7, 108.3)
- added J6: Conn_01x05_Pin, Connector_PinHeader_2.54mm:PinHeader_1x05_P2.54mm_Vertical, F.Cu at (69.7, 88.2)
- added R10: R, Resistor_SMD:R_0402_1005Metric, F.Cu at (77.1, 26.7)
- added R11: 1.5k, Resistor_SMD:R_0402_1005Metric, F.Cu at (77.1, 28.6)
- added R12: 10k, Resistor_SMD:R_0402_1005Metric, F.Cu at (77.1, 30.6)
- added R13: R, Resistor_SMD:R_0402_1005Metric, F.Cu at (77.1, 32.6)
- added R14: R, Resistor_SMD:R_0402_1005Metric, F.Cu at (80.0, 22.7)
- added R15: R, Resistor_SMD:R_0402_1005Metric, F.Cu at (80.0, 24.7)
- added R16: R, Resistor_SMD:R_0402_1005Metric, F.Cu at (80.0, 26.7)
- added R17: R, Resistor_SMD:R_0402_1005Metric, F.Cu at (80.0, 28.6)
- added R8: 10k, Resistor_SMD:R_0402_1005Metric, F.Cu at (77.1, 22.7)
- added R9: 10k, Resistor_SMD:R_0402_1005Metric, F.Cu at (77.1, 24.7)
- added S2: PTS815SJM250SMTR_LFS, SamacSys:PTS815SJM250SMTRLFS, F.Cu at (59.4, 61.4)
- added TH1: Thermistor, Resistor_SMD:R_0402_1005Metric, F.Cu at (80.0, 30.6)
- added U5: STM32F103C8T6, Package_QFP:LQFP-48_7x7mm_P0.5mm, F.Cu at (49.4, 80.2)
- C1, Cbst1, Ccomp1, Ccomp2, Cinx1, Cvcc1: footprint Capacitor_SMD:C_0603_1608Metric -> Capacitor_SMD:C_0402_1005Metric
- C4, Cin1, Cout1, Cout2, Cout3: footprint Capacitor_SMD:C_0603_1608Metric -> Capacitor_SMD:C_0805_2012Metric
- HSE1: value 8MHz -> 16MHz/16pF
- L1: value 2.2u -> 1.5u
- R1, R2, R3, R4, R5, R6, R7, Rcomp1, Rfbb1, Rfbt1: footprint Resistor_SMD:R_0603_1608Metric -> Resistor_SMD:R_0402_1005Metric
- moved HSE1 12.3 mm to (48.7, 71.2)
- moved L1 11.6 mm to (65.4, 72.6), turned to 0 degrees
- moved U7 8.44 mm to (64.4, 78.5), turned to 180 degrees
- moved C4 6.18 mm to (59.1, 76.4), turned to 180 degrees
- moved C3 4.80 mm to (59.1, 78.9), turned to 180 degrees
- moved S1 2.84 mm to (26.6, 100.2)
- moved U6 1.00 mm to (33.6, 96.3)
- moved PS1 0.59 mm to (73.6, 37.6)
- moved U2 0.40 mm to (80.2, 44.9)
Connections:
- C3 pad 1: V_SYS -> /EN3V3
- C4 pad 1: +3V3 -> +3.3V
- HSE1 pad 1: unconnected-(HSE1-Pad1) -> /OSC8M_IN
- HSE1 pad 3: unconnected-(HSE1-Pad3) -> Net-(C5-Pad1)
- J2 pad 4: /SCL -> /SCL1
- J2 pad 5: /SDA -> /SDA1
- R5 pad 2: /SCL -> /SCL1
- R6 pad 2: /SDA -> /SDA1
- S1 pad 1: unconnected-(S1-NC_1-Pad1) -> V_SYS
- S1 pad 2: unconnected-(S1-C_1-Pad2) -> /EN3V3
- S1 pad 5: +3V3_STM -> VDD
- S1 pad 6: +3V3 -> /EN3V3
- U1 pad 7: /SCL -> /SCL1
- U1 pad 8: /SDA -> /SDA1
- U2 pad 11: unconnected-(U2-TS-Pad11) -> Net-(U2-TS)
- U2 pad 13: unconnected-(U2-BAT_13-Pad13) -> +BATT
- U2 pad 14: unconnected-(U2-BAT_14-Pad14) -> +BATT
- U2 pad 17: unconnected-(U2-PGND_17-Pad17) -> GND
- U2 pad 18: unconnected-(U2-PGND_18-Pad18) -> GND
- U2 pad 22: unconnected-(U2-REGN-Pad22) -> /REGN
- U2 pad 25: unconnected-(U2-EXP-Pad25) -> GND
- U6 pad 1: unconnected-(U6-SDA-Pad1) -> /SDA1
- U6 pad 13: unconnected-(U6-ISET-Pad13) -> Net-(U6-ISET)
- U6 pad 14: unconnected-(U6-SCL-Pad14) -> /SCL1
- U6 pad 19: +3V3_STM -> +3.3V
- U6 pad 24: unconnected-(U6-IRQ-Pad24) -> /DISP_IRQ
- U6 pad 6: unconnected-(U6-GND-Pad6) -> GND
- U7 pad 1: +3V3 -> +3.3V
- U7 pad 10: +3V3 -> +3.3V
- U7 pad 5: V_SYS -> /EN3V3
- U7 pad 7: V_SYS -> /EN3V3
- U7 pad 8: V_SYS -> /EN3V3
Other:
- board text added: "BOOT"
- board text added: "GND"
- board text added: "RST"
- board text added: "RUN"
- board text added: "SWCLK"
- board text added: "SWDIO"
- board text added: "TRACE"
- board text added: "VDD"
- board text added: "VSYS"

Commit message: 14.08 save
Parts:
- removed Cbst1, Cinx1: 100n, Capacitor_SMD:C_0402_1005Metric
- removed Ccomp1: 39n, Capacitor_SMD:C_0402_1005Metric
- removed Ccomp2: 82p, Capacitor_SMD:C_0402_1005Metric
- removed Cin1: 10u, Capacitor_SMD:C_0805_2012Metric
- removed Cout1, Cout2, Cout3: 47u, Capacitor_SMD:C_0805_2012Metric
- removed Cvcc1: 2.2u, Capacitor_SMD:C_0402_1005Metric
- removed HSE1: 16MHz/16pF, Crystal:Crystal_SMD_3225-4Pin_3.2x2.5mm
- removed PS1: TPS25942ARVCT, SamacSys:QFN50P300X400X80-21N
- removed Rcomp1: 35.7k, Resistor_SMD:R_0402_1005Metric
- removed Rfbb1: 48.7k, Resistor_SMD:R_0402_1005Metric
- removed Rfbt1: 357k, Resistor_SMD:R_0402_1005Metric
- added C16: 1u, Capacitor_SMD:C_0402_1005Metric, F.Cu at (195.4, 63.5)
- added C17: 47n, Capacitor_SMD:C_0402_1005Metric, F.Cu at (200.7, 61.3)
- added C18: 8.2u, Capacitor_SMD:C_0603_1608Metric, F.Cu at (196.5, 61.5)
- added C19: 4.7u, Capacitor_SMD:C_0603_1608Metric, F.Cu at (199.3, 61.3)
- added C20: 10u, Capacitor_SMD:C_0603_1608Metric, F.Cu at (204.9, 66.1)
- added C21: 10u, Capacitor_SMD:C_0603_1608Metric, F.Cu at (206.5, 66.1)
- added C22: 10u, Capacitor_SMD:C_0805_2012Metric, F.Cu at (165.9, 36.7)
- added C23: 100n, Capacitor_SMD:C_0402_1005Metric, F.Cu at (167.6, 36.7)
- added C24: 2.2u, Capacitor_SMD:C_0402_1005Metric, F.Cu at (173.1, 34.6)
- added C25: 39n, Capacitor_SMD:C_0402_1005Metric, F.Cu at (178.2, 36.0)
- added C26: 82p, Capacitor_SMD:C_0402_1005Metric, F.Cu at (179.4, 36.0)
- added C27: 47u, Capacitor_SMD:C_0805_2012Metric, F.Cu at (180.5, 31.5)
- added C28: 47u, Capacitor_SMD:C_0805_2012Metric, F.Cu at (182.6, 31.5)
- added C29: 47u, Capacitor_SMD:C_0805_2012Metric, F.Cu at (184.7, 31.5)
- added C30: 100n, Capacitor_SMD:C_0402_1005Metric, F.Cu at (173.1, 30.4)
- added D4: Red, LED_SMD:LED_0402_1005Metric, F.Cu at (193.4, 68.4)
- added FB1: 120R, Resistor_SMD:R_0402_1005Metric, F.Cu at (130.9, 50.2)
- added L3: 1u, Inductor_SMD:L_6.3x6.3_H3, F.Cu at (206.1, 59.9)
- added R18: 10k, Resistor_SMD:R_0402_1005Metric, F.Cu at (130.9, 52.1)
- added R19: 470, Resistor_SMD:R_0402_1005Metric, F.Cu at (191.2, 69.6)
- added R20: 470, Resistor_SMD:R_0402_1005Metric, F.Cu at (191.2, 68.4)
- added R21: 10k, Resistor_SMD:R_0402_1005Metric, F.Cu at (130.9, 58.1)
- added R22: 1k, Resistor_SMD:R_0402_1005Metric, F.Cu at (153.6, 66.9)
- added R23: 35.7k, Resistor_SMD:R_0402_1005Metric, F.Cu at (177.0, 36.0)
- added R24: 357k, Resistor_SMD:R_0402_1005Metric, F.Cu at (174.4, 36.0)
- added R25: 48.7k, Resistor_SMD:R_0402_1005Metric, F.Cu at (175.6, 36.0)
- added S3: PTS815, SamacSys:PTS815SJM250SMTRLFS, F.Cu at (135.4, 67.5)
- added S4: PTS815, SamacSys:PTS815SJM250SMTRLFS, F.Cu at (135.4, 73.8)
- C2, C5: value 22p -> 100n
- J2: value Conn_01x05 -> Conn_01x05_Pin
- J5: value USB_B_Micro -> Conn_01x03_Pin; footprint Connector_USB:USB_Micro-B_Amphenol_10118193-0001LF_Horizontal -> Connector_PinHeader_2.54mm:PinHeader_1x03_P2.54mm_Vertical
- J6: value Conn_01x05_Pin -> Conn_01x03_Pin; footprint Connector_PinHeader_2.54mm:PinHeader_1x05_P2.54mm_Vertical -> Connector_PinHeader_2.54mm:PinHeader_1x03_P2.54mm_Vertical
- R10, R13: value R -> 10k
- R11: value 1.5k -> 10k
- R16: value R -> 5.25k
- R17: value R -> 31.23k
- R6: value 10k -> 158R
- R7: value 10k -> 1k
- S2: value PTS815SJM250SMTR_LFS -> PTS815
- moved U2 121.8 mm to (200.0, 66.6), turned to 0 degrees
- moved C15 115.9 mm to (204.0, 69.8), turned to -90 degrees
- moved D3 113.0 mm to (193.4, 69.5), turned to 180 degrees
- moved R16 112.1 mm to (186.8, 60.6)
- moved R17 112.1 mm to (186.8, 62.6)
- moved TH1 112.1 mm to (186.8, 64.6)
- moved R6 111.1 mm to (200.3, 70.8), turned to -90 degrees
- moved J5 97.4 mm to (113.8, 51.5)
- moved R10 84.7 mm to (153.6, 62.9)
- moved R11 84.7 mm to (153.6, 64.9)
- moved IC2 73.3 mm to (176.3, 31.5), turned to 90 degrees
- moved L2 69.3 mm to (168.7, 31.5), turned to 180 degrees
- moved R7 65.5 mm to (153.6, 60.9), turned to 0 degrees
- moved C2 61.3 mm to (118.0, 72.9)
- moved C5 61.3 mm to (118.0, 74.9)
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Connections:
- net +5V renamed +5V_OUT
- net Net-(IC2-SW_1) renamed /SW1
- net Net-(U2-TS) renamed /TS
- C2 pad 1: /OSC8M_IN -> /OFF
- C5 pad 1: Net-(C5-Pad1) -> /DISP
- D3 pad 1: Net-(D3-K) -> /PG
- D3 pad 2: +3.3V -> Net-(D3-A)
- IC2 pad 6: /EN5V0 -> /5VEN
- J2 pad 2: V_MCU_LOGIC -> /SWO
- J2 pad 3: /INT -> /SWCLK
- J2 pad 4: /SCL1 -> /SWDIO
- J2 pad 5: /SDA1 -> VDD
- J5 pad 1: VDD -> GND
- J5 pad 2: /USB- -> /RX
- J5 pad 3: /USB+ -> /TX
- J6 pad 2: /TRACESW -> /TRIG
- J6 pad 3: /SWCLK -> /REACT
- R10 pad 1: /OSC8M_OUT -> Net-(S3-NO1)
- R10 pad 2: Net-(C5-Pad1) -> GND
- R11 pad 1: +3.3V -> Net-(S4-NO1)
- R11 pad 2: /USB+ -> GND
- R13 pad 1: Net-(D3-K) -> +3.3V
- R13 pad 2: GND -> /INT_BQ
- R5 pad 1: V_MCU_LOGIC -> +3.3V
- R5 pad 2: /SCL1 -> /INT_MAX
- R6 pad 1: V_MCU_LOGIC -> /ILIM
- R6 pad 2: /SDA1 -> GND
- R7 pad 1: V_MCU_LOGIC -> Net-(S3-NO1)
- R7 pad 2: /INT -> /OFF
- S1 pad 5: VDD -> unconnected-(S1-NC_2-Pad5)
- S1 pad 7: unconnected-(S1-NO_2-Pad7) -> VDD
- U1 pad 5: /INT -> /INT_MAX
- U1 pad 7: /SCL1 -> /SCL
- U1 pad 8: /SDA1 -> /SDA
- U2 pad 1: unconnected-(U2-VBUS_1-Pad1) -> +5V_CHARGE
- U2 pad 10: unconnected-(U2-ILIM-Pad10) -> /ILIM
- U2 pad 15: unconnected-(U2-SYS_15-Pad15) -> V_SYS
- U2 pad 16: unconnected-(U2-SYS_16-Pad16) -> V_SYS
- U2 pad 19: unconnected-(U2-SW_19-Pad19) -> /SW2
- U2 pad 20: unconnected-(U2-SW_20-Pad20) -> /SW2
- U2 pad 21: unconnected-(U2-BTST-Pad21) -> /BTST
- U2 pad 23: unconnected-(U2-PMID-Pad23) -> /PMID
- U2 pad 24: unconnected-(U2-VBUS_24-Pad24) -> +5V_CHARGE
- U2 pad 3: unconnected-(U2-~{PG}-Pad3) -> /PG
- U2 pad 4: unconnected-(U2-STAT-Pad4) -> /STAT
- U2 pad 5: unconnected-(U2-SCL-Pad5) -> /SCL
- U2 pad 6: unconnected-(U2-SDA-Pad6) -> /SDA
- U2 pad 7: unconnected-(U2-INT-Pad7) -> /INT_BQ
- U2 pad 9: unconnected-(U2-~{CE}-Pad9) -> GND
- U5 pad 10: unconnected-(U5-PA0-Pad10) -> /OFF
- U5 pad 11: unconnected-(U5-PA1-Pad11) -> /OFF
- U5 pad 18: unconnected-(U5-PB0-Pad18) -> /DISP
- U5 pad 19: unconnected-(U5-PB1-Pad19) -> /REACT
- U5 pad 2: unconnected-(U5-PC13-Pad2) -> /LED
- U5 pad 20: unconnected-(U5-PB2-Pad20) -> /TRIG
- U5 pad 25: unconnected-(U5-PB12-Pad25) -> /5VEN
- U5 pad 30: unconnected-(U5-PA9-Pad30) -> /TX
- U5 pad 31: unconnected-(U5-PA10-Pad31) -> /RX
- U5 pad 32: /USB+ -> unconnected-(U5-PA11-Pad32)
- U5 pad 33: /USB- -> unconnected-(U5-PA12-Pad33)
- U5 pad 39: /TRACESW -> /SWO
- U5 pad 42: unconnected-(U5-PB6-Pad42) -> /SCL
- U5 pad 43: unconnected-(U5-PB7-Pad43) -> /SDA
- U5 pad 5: /OSC8M_IN -> unconnected-(U5-PD0-Pad5)
- U5 pad 6: /OSC8M_OUT -> unconnected-(U5-PD1-Pad6)
- U6 pad 1: /SDA1 -> /SDA
- U6 pad 14: /SCL1 -> /SCL
Routing:
- net Net-(IC2-COMP): track 0.00 -> 5.88 mm
- net Net-(IC2-VCC): track 0.00 -> 3.98 mm
- net Net-(IC2-FB_1): track 0.00 -> 3.85 mm
- net Net-(IC2-BST): track 0.00 -> 2.41 mm
- net Net-(C25-Pad1): track 0.00 -> 1.62 mm
- added copper zone on F.Cu, net +5V_OUT
- added copper zone on F.Cu, net /SW1
- added copper zone on In1.Cu, net GND
- added copper zone on F.Cu, net V_SYS
Other:
- copper layers 2 -> 4
- board text removed: "TRACE"

Commit message: PCB wersja 1.0 koniec
Parts:
- removed S1: JS202011JCQN, SamacSys:JS202011JCQN
- added C31: 100n, Capacitor_SMD:C_0402_1005Metric, F.Cu at (55.1, 75.1)
- added C32: 1u, Capacitor_SMD:C_0402_1005Metric, F.Cu at (51.7, 52.9)
- added C33: 100n, Capacitor_SMD:C_0402_1005Metric, F.Cu at (58.0, 74.7)
- added D5: Green, LED_SMD:LED_0402_1005Metric, F.Cu at (82.0, 40.8)
- added FID1: Fiducial, stencil_pin:stencil_pin, F.Cu at (24.8, 102.6)
- added FID2: Fiducial, stencil_pin:stencil_pin, F.Cu at (74.8, 102.6)
- added FID3: Fiducial, stencil_pin:stencil_pin, F.Cu at (24.8, 52.6)
- added G***: LOGO, logo:logo, B.Cu at (65.9, 62.1)
- added H1: MountingHole, MountingHole:MountingHole_2.2mm_M2, F.Cu at (106.8, 72.6)
- added H2: MountingHole, MountingHole:MountingHole_2.2mm_M2, F.Cu at (106.8, 34.6)
- added H3: MountingHole, MountingHole:MountingHole_2.2mm_M2, F.Cu at (94.8, 22.6)
- added H4: MountingHole, MountingHole:MountingHole_2.2mm_M2, F.Cu at (56.8, 22.6)
- added H5: MountingHole, MountingHole:MountingHole_2.2mm_M2, F.Cu at (22.8, 97.6)
- added H6: MountingHole, MountingHole:MountingHole_2.2mm_M2, F.Cu at (31.8, 106.6)
- added H7: MountingHole, MountingHole:MountingHole_2.2mm_M2, F.Cu at (27.8, 35.6)
- added H8: MountingHole, MountingHole:MountingHole_2.2mm_M2, F.Cu at (93.8, 101.6)
- added J7: 87583-0010RHLF, 87583-0010RHLF:AMPHENOL_87583-0010RHLF, F.Cu at (106.0, 85.9)
- added J8: SLW-66527511-SMT-TR, SamacSys:SLW66527511SMTTR, B.Cu at (108.0, 45.7)
- added J9: Conn_01x02, Connector_PinHeader_2.54mm:PinHeader_1x02_P2.54mm_Vertical, F.Cu at (96.1, 97.3)
- added JP1: SolderJumper_2_Open, Resistor_SMD:R_0805_2012Metric, F.Cu at (60.4, 72.6)
- added R26: 430, Resistor_SMD:R_0402_1005Metric, F.Cu at (80.2, 42.6)
- added R27: 10k, Resistor_SMD:R_0402_1005Metric, F.Cu at (96.0, 43.5)
- added R28: 10k, Resistor_SMD:R_0402_1005Metric, F.Cu at (96.8, 42.7)
- added R29: 10k, Resistor_SMD:R_0402_1005Metric, F.Cu at (56.7, 74.7)
- added TP1: TestPoint, TestPoint:TestPoint_Pad_1.0x1.0mm, F.Cu at (35.3, 34.4)
- added TP10: TestPoint, TestPoint:TestPoint_Pad_D3.0mm, F.Cu at (82.9, 84.6)
- added TP2: TestPoint, TestPoint:TestPoint_Pad_1.0x1.0mm, F.Cu at (75.4, 86.7)
- added TP3: TestPoint, TestPoint:TestPoint_Pad_1.0x1.0mm, F.Cu at (79.0, 77.6)
- added TP4: TestPoint, TestPoint:TestPoint_Pad_1.0x1.0mm, F.Cu at (42.8, 75.0)
- added TP5: TestPoint, TestPoint:TestPoint_Pad_1.0x1.0mm, F.Cu at (72.1, 69.6)
- added TP6: TestPoint, TestPoint:TestPoint_Pad_1.0x1.0mm, F.Cu at (61.8, 62.0)
- added TP7: TestPoint, TestPoint:TestPoint_Pad_1.0x1.0mm, F.Cu at (72.7, 76.7)
- added TP8: TestPoint, TestPoint:TestPoint_Pad_1.0x1.0mm, F.Cu at (92.7, 52.7)
- added TP9: TestPoint, TestPoint:TestPoint_Pad_1.0x1.0mm, F.Cu at (94.9, 52.7)
- J2: value Conn_01x05_Pin -> Conn_01x05; footprint Connector_PinHeader_2.54mm:PinHeader_1x05_P2.54mm_Vertical -> Connector_PinSocket_2.54mm:PinSocket_1x05_P2.54mm_Vertical
- J3: moved to B.Cu
- J5: value Conn_01x03_Pin -> Conn_01x05; footprint Connector_PinHeader_2.54mm:PinHeader_1x03_P2.54mm_Vertical -> Connector_PinSocket_2.54mm:PinSocket_1x05_P2.54mm_Vertical
- J6: value Conn_01x03_Pin -> Conn_01x02; footprint Connector_PinHeader_2.54mm:PinHeader_1x03_P2.54mm_Vertical -> Connector_PinHeader_2.54mm:PinHeader_1x02_P2.54mm_Vertical
- L1: footprint Inductor_SMD:L_6.3x6.3_H3 -> Inductor_SMD:L_1008_2520Metric
- L3: footprint Inductor_SMD:L_6.3x6.3_H3 -> IHLP2020ABER1R0M01:IND_R2M01_VIS
- R14: value R -> 430
- TH1: value Thermistor -> B25/85 3435K; footprint Resistor_SMD:R_0402_1005Metric -> Resistor_SMD:R_0805_2012Metric
- moved C15 158.9 mm to (45.3, 62.5), turned to 180 degrees
- moved C21 157.5 mm to (49.0, 65.0), turned to 0 degrees
- moved R6 156.7 mm to (44.2, 57.5), turned to 180 degrees
- moved C20 155.9 mm to (49.0, 63.4), turned to 0 degrees
- moved U2 151.8 mm to (48.5, 58.5), turned to -90 degrees
- moved L3 151.1 mm to (55.1, 64.7), turned to 90 degrees
- moved D4 147.8 mm to (46.5, 52.2), turned to 90 degrees
- moved C17 147.2 mm to (53.5, 59.9), turned to 0 degrees
- moved D3 146.6 mm to (47.8, 52.2), turned to 90 degrees
- moved R20 145.9 mm to (46.5, 49.5), turned to 90 degrees
- moved C19 145.6 mm to (53.7, 58.2), turned to 0 degrees
- moved R19 144.8 mm to (47.8, 49.5), turned to 90 degrees
- moved C16 144.0 mm to (51.7, 54.1), turned to 0 degrees
- moved C18 143.1 mm to (53.5, 55.3), turned to 90 degrees
- moved R16 142.8 mm to (44.0, 60.3), turned to 180 degrees
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Connections:
- net /EN3V3 renamed /VIN_STM
- net /OFF renamed /ON/OFF
- D1 pad 1: Net-(D1-K) -> GND
- D1 pad 2: +5V_CHARGE -> Net-(D1-A)
- D2 pad 1: Net-(D2-K) -> GND
- D2 pad 2: +5V_OUT -> Net-(D2-A)
- J2 pad 1: GND -> /TX
- J2 pad 2: /SWO -> /RX
- J2 pad 3: /SWCLK -> /REACT
- J2 pad 4: /SWDIO -> /TRIG
- J2 pad 5: VDD -> GND
- J5 pad 1: GND -> VDD
- J5 pad 2: /RX -> /SWO
- J5 pad 3: /TX -> /SWCLK
- J6 pad 1: GND -> +3.3V
- J6 pad 2: /TRIG -> /O/X
- R1 pad 1: Net-(J4-CC1) -> GND
- R1 pad 2: GND -> Net-(J4-CC1)
- R10 pad 1: Net-(S3-NO1) -> /O/X
- R14 pad 1: Net-(D1-K) -> +5V_CHARGE
- R14 pad 2: GND -> Net-(D1-A)
- R15 pad 1: Net-(D2-K) -> +5V_OUT
- R15 pad 2: GND -> Net-(D2-A)
- R2 pad 1: Net-(J4-CC2) -> GND
- R2 pad 2: GND -> Net-(J4-CC2)
- R7 pad 1: Net-(S3-NO1) -> /O/X
- S3 pad 3: Net-(S3-NO1) -> /O/X
- S3 pad 4: Net-(S3-NO1) -> /O/X
- U5 pad 13: unconnected-(U5-PA3-Pad13) -> /INT_BQ
- U5 pad 14: unconnected-(U5-PA4-Pad14) -> /INT_MAX
Routing:
- net +3.3V: track 0.00 -> 302.1 mm, vias 0 -> 8
- net /SDA: track 0.00 -> 147.8 mm, vias 0 -> 4
- net /SCL: track 0.00 -> 146.0 mm, vias 0 -> 4
- net V_SYS: track 0.00 -> 124.7 mm, vias 0 -> 1
- net +5V_OUT: track 0.00 -> 110.5 mm
- net GND: track 0.00 -> 92.1 mm, vias 0 -> 558
- net /5VEN: track 0.00 -> 86.8 mm
- net +BATT: track 0.00 -> 85.1 mm, vias 0 -> 14
- net /segE: track 0.00 -> 80.2 mm
- net /segDP: track 0.00 -> 79.6 mm, vias 0 -> 1
- net /segC: track 0.00 -> 78.3 mm
- net /segG: track 0.00 -> 78.2 mm
- net /segD: track 0.00 -> 78.0 mm, vias 0 -> 1
- net /segA: track 0.00 -> 76.1 mm, vias 0 -> 1
- net /segF: track 0.00 -> 75.2 mm, vias 0 -> 1
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- added copper zone on F.Cu, net +3.3V
- added copper zone on F.Cu, net +5V_CHARGE
- added copper zone on B.Cu, net +BATT
- added copper zone on F.Cu, net +BATT
- added copper zone on F.Cu, net /PMID
- added copper zone on F.Cu, net /SW2
- added copper zone on F.Cu, net /VIN_STM
- added copper zone on B.Cu, net GND
- added copper zone on F.Cu, net GND
- added copper zone on In2.Cu, net GND
- added copper zone on F.Cu, net Net-(U7-L1)
- added copper zone on F.Cu, net Net-(U7-L2)
Other:
- outline, holes or cut-outs redrawn
- board text added: "+"
- board text added: "-"
- board text added: "3V3"
- board text added: "5V CHARGE"
- board text added: "5V OUT"
- board text added: "5VEN"
- board text added: "CHARGER INPUT"
- board text added: "CLK"
- board text added: "DIO"
- board text added: "DISPLAY"
- board text added: "O/X BTN"
- board text added: "ON-OFF"
- board text added: "REACT"
- board text added: "RESET"
- board text added: "RPI OUTPUT"
- board text added: "RPI-G"
- board text added: "RX"
- board text added: "SW-G"
- board text added: "SWO"
- board text added: "TRIG"
- board text added: "TX"
- board text added: "Toggle MCU boot/run"
- board text added: "Toggle MCU pwr src"
- board text added: "V STM"
- board text added: "VBAT"
- board text added: "https://github.com/SzymonGogulski"
- board text removed: "RST"
- board text removed: "SWCLK"
- board text removed: "SWDIO"
