File: BQ2xxxx/BQ2xxxx.kicad_sch (KiCad schematic)
At the start: 8 parts, among them J1 1054500101, J2 1054500101, U1 BQ25895MRTWT, U2 BQ24296MRGER

Commit message: MAIN: 25.06.2025
Parts:
- removed +5V, GND: TestPoint, TestPoint:TestPoint_Pad_D3.0mm, symbol Connector:TestPoint
- removed J1, J2: 1054500101, 1054500101:MOLEX_1054500101, symbol 1054500101:1054500101
- removed U1: BQ25895MRTWT, BQ25895MRTWT:QFN50P400X400X80-25N, symbol BQ25895MRTWT:BQ25895MRTWT
- added C1: 0.1u, Capacitor_SMD:C_0603_1608Metric, symbol Device:C
- added C3, Cin1: 10u, Capacitor_SMD:C_0603_1608Metric, symbol Device:C
- added C4: 33u, Capacitor_SMD:C_0603_1608Metric, symbol Device:C
- added Cbst1, Cinx1: 100n, Capacitor_SMD:C_0603_1608Metric, symbol Device:C
- added Ccomp1: 39n, Capacitor_SMD:C_0603_1608Metric, symbol Device:C
- added Ccomp2: 82p, Capacitor_SMD:C_0603_1608Metric, symbol Device:C
- added Cout1, Cout2, Cout3: 47u, Capacitor_SMD:C_0603_1608Metric, symbol Device:C
- added Cvcc1: 2.2u, Capacitor_SMD:C_0603_1608Metric, symbol Device:C
- added HSE1: 8MHz, Crystal:Crystal_SMD_3225-4Pin_3.2x2.5mm, symbol Device:Crystal_GND24
- added IC1: STM32F030R8T6, STM32F030R8T6:QFP50P1200X1200X160-64N, symbol STM32F030R8T6:STM32F030R8T6
- added IC2: TPS61288RQQR, SamacSys:TPS61288RQQR, symbol SymacSys:TPS61288RQQR
- added J1, J4: USB4125-GF-A, SamacSys:USB4125GFA, symbol SymacSys:USB4125-GF-A
- added J2: Conn_01x05, Connector_PinHeader_2.54mm:PinHeader_1x05_P2.54mm_Vertical, symbol Connector_Generic:Conn_01x05
- added L1: 2.2u, Inductor_SMD:L_6.3x6.3_H3, symbol Device:L
- added L2: 1.5u, Inductor_SMD:L_6.3x6.3_H3, symbol Device:L
- added LSE1: 32.768kHz, Crystal:Crystal_SMD_3215-2Pin_3.2x1.5mm, symbol Device:Crystal
- added PS1: TPS25942ARVCT, SamacSys:QFN50P300X400X80-21N, symbol SymacSys:TPS25942ARVCT
- added R1, R2: 5.1k, Resistor_SMD:R_0603_1608Metric, symbol Device:R
- added R3, R4, R5, R6, R7: 10k, Resistor_SMD:R_0603_1608Metric, symbol Device:R
- added Rcomp1: 35.7k, Resistor_SMD:R_0603_1608Metric, symbol Device:R
- added Rfbb1: 48.7k, Resistor_SMD:R_0603_1608Metric, symbol Device:R
- added Rfbt1: 357k, Resistor_SMD:R_0603_1608Metric, symbol Device:R
- added S1: JS202011JCQN, SamacSys:JS202011JCQN, symbol SymacSys:JS202011JCQN
- added U1: MAX17048G_T10, MAX17048G_T10:SON50P200X200X80-9N, symbol MAX17048G+T10:MAX17048G_T10
- added U3, U4: CC56-12GWA, Display_7Segment:CC56-12GWA, symbol Display_Character:CC56-12GWA
- added U6: AS1115-BSST, Package_SO:QSOP-24_3.9x8.7mm_P0.635mm, symbol Interface_Expansion:AS1115-BSST
- added U7: TPS63001, Package_SON:Texas_DRC0010J, symbol Regulator_Switching:TPS63001
Connections:
- net +BATT: now also C1.1, U1.2 (CELL), U1.3 (VDD)
- net GND: now also C1.2, C3.2, C4.2, Ccomp1.2, Ccomp2.2, Cin1.1, Cinx1.2, Cout1.2, Cout2.2, Cout3.2, Cvcc1.2, HSE1.2, HSE1.4, IC2.10 (AGND), IC2.13 (PGND_2), IC2.3 (PGND_1), J1.A12 (GND_1), J1.B12 (GND_2), J1.MH1 (SH1), J1.MH2 (SH2), J1.MH3 (SH3), J1.MH4 (SH4), J2.1 (Pin_1), J4.A12 (GND_1), J4.B12 (GND_2), J4.MH1 (SH1), J4.MH2 (SH2), J4.MH3 (SH3), J4.MH4 (SH4), R1.2, R2.2, Rfbb1.2, U1.1 (CTG), U1.4 (GND), U1.6 (QSTRT), U1.9 (EP), U7.11 (PGND), U7.3 (PGND), U7.9 (GND)
- new net: Cbst1.2, IC2.4 (SW_1), IC2.9 (SW_2), L2.1
- new net: IC2.1 (FB_1), IC2.12 (FB_2), Rfbb1.1, Rfbt1.2
- new net: Ccomp2.1, IC2.2 (COMP), Rcomp1.1
- new net: J4.B5 (CC2), R2.1
- new net: Cvcc1.1, IC2.11 (VCC)
- new net: J1.A5 (CC1), R4.2
- new net: L1.1, U7.2 (L2)
- new net: L1.2, U7.4 (L1)
- new net: Cbst1.1, IC2.8 (BST)
- new net: J4.A5 (CC1), R1.1
- new net: Ccomp1.1, Rcomp1.2
- new net: J1.B5 (CC2), R3.2
- new net +3V3: C4.1, S1.6 (C_2), U7.1 (VOUT), U7.10 (FB)
- new net +3V3_STM: S1.5 (NC_2), U6.19 (VDD)
- new net +5V: Cout1.1, Cout2.1, Cout3.1, IC2.14 (VOUT_2), IC2.5 (VOUT_1), J1.A9 (VBUS_1), J1.B9 (VBUS_2), R3.1, R4.1, Rfbt1.1
- new net +5V_CHARGE: J4.A9 (VBUS_1), J4.B9 (VBUS_2)
- new net Digit0: U3.12 (CC1), U6.2 (DIG0)
- new net Digit1: U3.9 (CC2), U6.3 (DIG1)
- new net Digit2: U3.8 (CC3), U6.4 (DIG2)
- new net Digit3: U3.6 (CC4), U6.5 (DIG3)
- new net Digit4: U4.12 (CC1), U6.7 (DIG4)
- new net Digit5: U4.9 (CC2), U6.8 (DIG5)
- new net Digit6: U4.8 (CC3), U6.9 (DIG6)
- new net Digit7: U4.6 (CC4), U6.10 (DIG7)
- new net EN3V3: U7.6 (EN)
- new net EN5V0: IC2.6 (EN)
- new net INT: J2.3 (Pin_3), R7.2, U1.5 (~{ALERT})
- new net SCL: J2.4 (Pin_4), R5.2, U1.7 (SCL)
- new net SDA: J2.5 (Pin_5), R6.2, U1.8 (SDA)
- new net V_MCU_LOGIC: J2.2 (Pin_2), R5.1, R6.1, R7.1
- new net V_SYS: C3.1, Cin1.2, Cinx1.1, IC2.15 (VIN_2), IC2.7 (VIN_1), L2.2, U7.5 (VIN), U7.7 (PS/SYNC), U7.8 (VINA)
- new net segA: U3.11 (a), U4.11 (a), U6.15 (SEGA)
- new net segB: U3.7 (b), U4.7 (b), U6.17 (SEGB)
- new net segC: U3.4 (c), U4.4 (c), U6.20 (SEGC)
- new net segD: U3.2 (d), U4.2 (d), U6.23 (SEGD)
- new net segDP: U3.3 (DPX), U4.3 (DPX), U6.22 (SEGDP)
- new net segE: U3.1 (e), U4.1 (e), U6.21 (SEGE)
- new net segF: U3.10 (f), U4.10 (f), U6.16 (SEGF)
- new net segG: U3.5 (g), U4.5 (g), U6.18 (SEGG)
- no-connect marks 1 -> 5
Other:
- note added: "BOOST VBAT -> 5.0V"
- note added: "BQ24296 / Efuse"
- note added: "BUCKBOOST VBAT -> 3.3V"
- note added: "Battery Holder"
- note added: "CELL FUEL GAUGE"
- note added: "GOLD PIN CONNECTOR"
- note added: "NOTES Common Cathode Displays"
- note added: "PULLUP RESISTORS"
- note added: "SPI 8-digit 7-segment display"
- note added: "STM32"
- note added: "STM32/Display ON/OFF"
- note added: "USB-C Sink"
- note added: "USB-C Source"
- note removed: "BQ24296"
- note removed: "BQ25895"
- note removed: "Battery Holder / MAX17048"
- note removed: "CONVERTERS 5.0V"
- note removed: "IN"
- note removed: "MAX17048"
- note removed: "OUT / Efuse"
- note removed: "https://www.digikey.pl/pl/articles/an-overview-of-usb-type-c-in-power-only-designs"
- moved on the sheet: BT1, BT2, U2

Commit message: Work in progress: Schematic
Parts:
- removed IC1: STM32F030R8T6, STM32F030R8T6:QFP50P1200X1200X160-64N, symbol STM32F030R8T6:STM32F030R8T6
- removed LSE1: 32.768kHz, Crystal:Crystal_SMD_3215-2Pin_3.2x1.5mm, symbol Device:Crystal
- added C10, C15: 10u, Capacitor_SMD:C_0603_1608Metric, symbol Device:C
- added C11: 10n, Capacitor_SMD:C_0402_1005Metric, symbol Device:C
- added C12, C13: 1u, Capacitor_SMD:C_0402_1005Metric, symbol Device:C
- added C14, C6, C7, C8, C9: 100n, Capacitor_SMD:C_0402_1005Metric, symbol Device:C
- added C16: 1u, symbol Device:C
- added C17: 47n, symbol Device:C
- added C2, C5: 22p, Capacitor_SMD:C_0402_1005Metric, symbol Device:C
- added D1, D2: Blue, LED_SMD:LED_0402_1005Metric, symbol Device:LED
- added D3, D4: LED, symbol Device:LED
- added FB1: 120R, symbol Device:FerriteBead
- added J3: SLW-66527511-SMT-TR, SamacSys:SLW66527511SMTTR, symbol SymacSys:SLW-66527511-SMT-TR
- added J5: USB_B_Micro, Connector_USB:USB_Micro-B_Amphenol_10118193-0001LF_Horizontal, symbol Connector:USB_B_Micro
- added J7: Conn_01x04_Pin, symbol Connector:Conn_01x04_Pin
- added L3: L, symbol Device:L
- added R10, R14, R15, R16, R17: R, Resistor_SMD:R_0402_1005Metric, symbol Device:R
- added R11: 1.5k, Resistor_SMD:R_0402_1005Metric, symbol Device:R
- added R12, R8, R9: 10k, Resistor_SMD:R_0402_1005Metric, symbol Device:R
- added R13, R18: 10k, symbol Device:R
- added R19, R20: 470, symbol Device:R
- added S2: PTS815SJM250SMTR_LFS, SamacSys:PTS815SJM250SMTRLFS, symbol SymacSys:PTS815SJM250SMTR_LFS
- added TH1: Thermistor, Resistor_SMD:R_0402_1005Metric, symbol Device:Thermistor
- added U5: STM32F103C8T6, Package_QFP:LQFP-48_7x7mm_P0.5mm, symbol MCU_ST_STM32F1:STM32F103C8Tx
- C1, Cbst1, Ccomp1, Ccomp2, Cinx1, Cvcc1: footprint Capacitor_SMD:C_0603_1608Metric -> Capacitor_SMD:C_0402_1005Metric
- C4, Cin1, Cout1, Cout2, Cout3: footprint Capacitor_SMD:C_0603_1608Metric -> Capacitor_SMD:C_0805_2012Metric
- HSE1: value 8MHz -> 16MHz/16pF
- L1: value 2.2u -> 1.5u
- R1, R2, R3, R4, R5, R6, R7, Rcomp1, Rfbb1, Rfbt1: footprint Resistor_SMD:R_0603_1608Metric -> Resistor_SMD:R_0402_1005Metric
Connections:
- net +5V_CHARGE: now also U2.1 (VBUS_1), U2.24 (VBUS_24), C16.1, D1.2 (A)
- net +BATT: now also U2.13 (BAT_13), U2.14 (BAT_14), C15.1
- net EN3V3: now also C3.1, S1.2 (C_1), S1.6 (C_2), U7.5 (VIN), U7.7 (PS/SYNC), U7.8 (VINA)
- net GND: now also U2.17 (PGND_17), U2.18 (PGND_18), U2.25 (EXP), U2.9 (~{CE}), U6.6 (GND), C10.2, C11.2, C12.2, C13.2, C14.2, C15.2, C16.2, C2.2, C5.2, C6.2, C7.2, C8.2, C9.2, J3.1, J3.MP1, J3.MP2, J3.MP3, J3.MP4, J5.5 (GND), J5.6 (Shield), J7.1 (Pin_1), R14.2, R15.2, R17.2, S2.3 (NO_1), S2.4 (NO_2), TH1.2, U5.23 (VSS), U5.35 (VSS), U5.47 (VSS), U5.8 (VSSA)
- net V_SYS: now also S1.1 (NC_1), U2.15 (SYS_15), U2.16 (SYS_16), R19.2, R20.2; no longer C3.1, U7.5 (VIN), U7.7 (PS/SYNC), U7.8 (VINA)
- net OSC8M_IN: now reaches HSE1.1
- net OSC8M_IN: now also C2.1, U5.5 (PD0)
- net at HSE1.3: now also C5.1, R10.2
- net SDA STM: now reaches U6.1 (SDA)
- net SDA STM: now also U2.6 (SDA), R18.2
- net at U6.13 (ISET): now also R8.2
- net SCL STM: now reaches U6.14 (SCL)
- net SCL STM: now also U2.5 (SCL), R13.2
- net DISP_IRQ: now reaches U6.24 (IRQ)
- net TS: now reaches U2.11 (TS)
- net TS: now also R16.2, R17.1, TH1.1
- net at U2.19 (SW_19): now also U2.20 (SW_20), C17.1, L3.1
- net at U2.21 (BTST): now also C17.2
- net REGN: now reaches U2.22 (REGN)
- net REGN: now also R16.1
- net PG: now reaches U2.3 (~{PG})
- net PG: now also D3.1 (K)
- net STAT: now reaches U2.4 (STAT)
- net STAT: now also D4.1 (K)
- net +3V3 renamed +3.3V
- net +3.3V: now also U6.19 (VDD), C10.1, C13.1, C6.1, C7.1, C8.1, C9.1, FB1.2, J3.3, R11.1, R12.1, R13.1, R18.1, R8.1, U5.1 (VBAT), U5.24 (VDD), U5.36 (VDD), U5.48 (VDD); no longer S1.6 (C_2)
- net +3V3_STM renamed VDD
- net VDD: now also J5.1 (VBUS), J7.4 (Pin_4); no longer U6.19 (VDD)
- net +5V renamed +5V_OUT
- net +5V_OUT: now also D2.2 (A)
- net SCL renamed SCL1
- net SCL1: no longer U1.7 (SCL)
- net SDA renamed SDA1
- net SDA1: no longer U1.8 (SDA)
- new net: J3.2, R9.1
- new net: D3.2 (A), R19.1
- new net: D4.2 (A), R20.1
- new net: D1.1 (K), R14.1
- new net: D2.1 (K), R15.1
- new net +3.3VA: C11.1, C12.1, FB1.1, U5.9 (VDDA)
- new net BOOT: R9.2, U5.44 (BOOT0)
- new net NRST: C14.1, R12.2, S2.1 (COM_1), S2.2 (COM_2), U5.7 (NRST)
- new net OSC8M_OUT: R10.1, U5.6 (PD1)
- new net SCL RPI: U1.7 (SCL)
- new net SDA RPI: U1.8 (SDA)
- new net SWCLK: J7.2 (Pin_2), U5.37 (PA14)
- new net SWDIO: J7.3 (Pin_3), U5.34 (PA13)
- new net USB+: J5.3 (D+), R11.2, U5.32 (PA11)
- new net USB-: J5.2 (D-), U5.33 (PA12)
- no-connect marks 5 -> 4
Other:
- note added: "16MHz crystal"
- note added: "BUCKBOOST VSYS/VDD -> 3.3V"
- note added: "NOTATKI Wspólna katoda W R8 wypróbuj 10k, 20k, 25k"
- note added: "Reset button"
- note added: "SWD"
- note added: "Toggle BOOT/RUN"
- note added: "Toggle MCU power src"
- note removed: "BUCKBOOST VBAT -> 3.3V"
- note removed: "NOTES Common Cathode Displays"
- note removed: "STM32/Display ON/OFF"
- moved on the sheet: BT1, BT2, C1, Cbst1, Ccomp1, Ccomp2, Cin1, Cinx1, Cout1, Cout2, Cout3, Cvcc1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

Commit message: 14.08 save
Parts:
- removed HSE1: 16MHz/16pF, Crystal:Crystal_SMD_3225-4Pin_3.2x2.5mm, symbol Device:Crystal_GND24
- removed J2: Conn_01x05, Connector_PinHeader_2.54mm:PinHeader_1x05_P2.54mm_Vertical, symbol Connector_Generic:Conn_01x05
- removed J5: USB_B_Micro, Connector_USB:USB_Micro-B_Amphenol_10118193-0001LF_Horizontal, symbol Connector:USB_B_Micro
- removed J7: Conn_01x04_Pin, symbol Connector:Conn_01x04_Pin
- removed PS1: TPS25942ARVCT, SamacSys:QFN50P300X400X80-21N, symbol SymacSys:TPS25942ARVCT
- added C18: 8.2u, Capacitor_SMD:C_0603_1608Metric, symbol Device:C
- added C19: 4.7u, Capacitor_SMD:C_0603_1608Metric, symbol Device:C
- added C20, C21: 10u, Capacitor_SMD:C_0603_1608Metric, symbol Device:C
- added J2: Conn_01x05_Pin, Connector_PinHeader_2.54mm:PinHeader_1x05_P2.54mm_Vertical, symbol Connector:Conn_01x05_Pin
- added J5, J6: Conn_01x03_Pin, Connector_PinHeader_2.54mm:PinHeader_1x03_P2.54mm_Vertical, symbol Connector:Conn_01x03_Pin
- added R21: 10k, Resistor_SMD:R_0402_1005Metric, symbol Device:R
- added R22: 1k, Resistor_SMD:R_0402_1005Metric, symbol Device:R
- added S3, S4: PTS815, PTS815SJM250SMTRLFS, symbol SymacSys:PTS815SJM250SMTR_LFS
- C16, C17: footprint (none) -> Capacitor_SMD:C_0402_1005Metric
- C2, C5: value 22p -> 100n
- D3: value LED -> Green; footprint (none) -> LED_SMD:LED_0402_1005Metric
- D4: value LED -> Red; footprint (none) -> LED_SMD:LED_0402_1005Metric
- FB1, R13, R18, R19, R20: footprint (none) -> Resistor_SMD:R_0402_1005Metric
- L3: value L -> 1u; footprint (none) -> Inductor_SMD:L_6.3x6.3_H3
- R10: value R -> 10k
- R11: value 1.5k -> 10k
- R16: value R -> 5.25k
- R17: value R -> 31.23k
- R6: value 10k -> 158R
- R7: value 10k -> 1k
- S2: value PTS815SJM250SMTR_LFS -> PTS815
- renumbered Cin1 to C22, Cinx1 to C23, Cvcc1 to C24, Ccomp1 to C25, Ccomp2 to C26, Cout1 to C27, Cout2 to C28, Cout3 to C29, Cbst1 to C30, Rcomp1 to R23, Rfbt1 to R24, Rfbb1 to R25
Connections:
- net EN5V0 is gone; now on net 5VEN: IC2.6 (EN)
- net SCL RPI is gone; now on net SCL: U1.7 (SCL)
- net SCL1 is gone; now on net INT_MAX: R5.2
- net SDA RPI is gone; now on net SDA: U1.8 (SDA)
- net SDA STM is gone; now on net SDA: R18.2, U2.6 (SDA), U6.1 (SDA)
- net SDA1 is gone; now on net GND: R6.2
- net +3.3V: now also R5.1, R21.1, S3.1 (C1), S3.2 (C2), S4.1 (C1), S4.2 (C2); no longer R11.1
- net GND: now also R10.2, R11.2, C18.2, C19.2, C20.2, C21.2, J2.1 (Pin_1), J5.1 (Pin_1), J6.1 (Pin_1)
- net REGN: now also C19.1
- net SWCLK: now also J2.3 (Pin_3)
- net SWDIO: now also J2.4 (Pin_4)
- net VDD: now also S1.7 (NO_2), J2.5 (Pin_5); no longer S1.5 (NC_2)
- net V_SYS: now also L3.1, C20.1, C21.1
- net SW1: now reaches C30.2, IC2.4 (SW_1), IC2.9 (SW_2), L2.1
- net DISP: now reaches C5.1
- net DISP: now also U5.18 (PB0), R22.2; no longer R10.2
- net OFF: now reaches U5.10 (PA0)
- net OFF: now also C2.1, R7.2, U5.11 (PA1)
- net REACT: now reaches U5.19 (PB1)
- net REACT: now also J6.3 (Pin_3)
- net LED: now reaches U5.2 (PC13)
- net TRIG: now reaches U5.20 (PB2)
- net TRIG: now also J6.2 (Pin_2)
- net 5VEN: now reaches U5.25 (PB12)
- net TX: now reaches U5.30 (PA9)
- net TX: now also J5.3 (Pin_3)
- net RX: now reaches U5.31 (PA10)
- net RX: now also J5.2 (Pin_2)
- net SWO: now reaches U5.39 (PB3)
- net SWO: now also J2.2 (Pin_2)
- net SCL: now reaches U5.42 (PB6)
- net SCL: now also U2.5 (SCL), U6.14 (SCL), R21.2
- net SDA: now reaches U5.43 (PB7)
- net SW2: now reaches C17.1, U2.19 (SW_19), U2.20 (SW_20)
- net SW2: now also L3.2; no longer L3.1
- net BTST: now reaches C17.2, U2.21 (BTST)
- net ILIM: now reaches U2.10 (ILIM)
- net ILIM: now also R6.1
- net PMID: now reaches U2.23 (PMID)
- net PMID: now also C18.1
- net INT_BQ: now reaches U2.7 (INT)
- net INT_BQ: now also R13.2
- net INT renamed INT_MAX
- net INT_MAX: no longer R7.2
- net OSC8M_IN: no longer names the net of U5.5 (PD0)
- net OSC8M_IN: no longer C2.1
- net OSC8M_OUT: no longer names the net of R10.1
- net OSC8M_OUT: now also R7.1, S3.3 (NO1), S3.4 (NO2); no longer U5.6 (PD1)
- removed net SCL STM: R13.2, U2.5 (SCL), U6.14 (SCL)
- net USB+: no longer names the net of U5.32 (PA11)
- net USB+: no longer R11.2
- net USB-: no longer names the net of U5.33 (PA12)
- removed net V_MCU_LOGIC: R5.1, R6.1, R7.1
- new net: R11.1, R22.1, S4.3 (NO1), S4.4 (NO2)
Other:
- note added: "- czy gpio REACT/TRIG potrzebuje pull-up pull-down? - czy UART TX/RX potrezbuje pull-up pull-down? - DISP_IRQ/INT_MAX/INT_BQ wtf???"
- note added: "1-2 -> RUN 2-3 -> BOOT"
- note added: "DISP button"
- note added: "I2C 8-digit 8-segment display"
- note added: "IRQ/I2C PULLUPS"
- note added: "LED"
- note added: "ON/OFF button"
- note added: "REACT/TRIG"
- note added: "Toggle MCU power src (!!!!!!!!! WTF??) Chyba symbol/footprint jest nie ok"
- note added: "UART"
- note added: "USB-C Sink 5V@3A"
- note added: "USB-C Source 5V@3A"
- note added: "WTF?"
- note removed: "16MHz crystal"
- note removed: "GOLD PIN CONNECTOR"
- note removed: "PULLUP RESISTORS"
- note removed: "SPI 8-digit 7-segment display"
- note removed: "Toggle MCU power src"
- note removed: "USB-C Sink"
- note removed: "USB-C Source"
- moved on the sheet: BT1, BT2, C1, C10, C11, C12, C13, C14, C15, C16, C17, C3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

Commit message: PCB wersja 1.0 koniec
Parts:
- removed J2: Conn_01x05_Pin, Connector_PinHeader_2.54mm:PinHeader_1x05_P2.54mm_Vertical, symbol Connector:Conn_01x05_Pin
- removed J5, J6: Conn_01x03_Pin, Connector_PinHeader_2.54mm:PinHeader_1x03_P2.54mm_Vertical, symbol Connector:Conn_01x03_Pin
- removed S1: JS202011JCQN, SamacSys:JS202011JCQN, symbol SymacSys:JS202011JCQN
- removed U1: MAX17048G_T10, MAX17048G_T10:SON50P200X200X80-9N, symbol MAX17048G+T10:MAX17048G_T10
- added C31, C33: 100n, Capacitor_SMD:C_0402_1005Metric, symbol Device:C
- added C32: 1u, Capacitor_SMD:C_0402_1005Metric, symbol Device:C
- added D5: Green, LED_SMD:LED_0402_1005Metric, symbol Device:LED
- added FID1, FID2, FID3: Fiducial, stencil_pin:stencil_pin, symbol Mechanical:Fiducial
- added H1, H2, H3, H4, H5, H6, H7, H8: MountingHole, MountingHole:MountingHole_2.2mm_M2, symbol Mechanical:MountingHole
- added J2, J5: Conn_01x05, Connector_PinSocket_2.54mm:PinSocket_1x05_P2.54mm_Vertical, symbol Connector_Generic:Conn_01x05
- added J6, J9: Conn_01x02, Connector_PinHeader_2.54mm:PinHeader_1x02_P2.54mm_Vertical, symbol Connector_Generic:Conn_01x02
- added J7: 87583-0010RHLF, 87583-0010RHLF:AMPHENOL_87583-0010RHLF, symbol 87583-0010RHLF:87583-0010RHLF
- added J8: SLW-66527511-SMT-TR, SamacSys:SLW66527511SMTTR, symbol SymacSys:SLW-66527511-SMT-TR
- added JP1: SolderJumper_2_Open, Resistor_SMD:R_0805_2012Metric, symbol Jumper:SolderJumper_2_Open
- added R26: 430, Resistor_SMD:R_0402_1005Metric, symbol Device:R
- added R27, R28, R29: 10k, Resistor_SMD:R_0402_1005Metric, symbol Device:R
- added TP1, TP2, TP3, TP4, TP5, TP6, TP7, TP8, TP9: TestPoint, TestPoint:TestPoint_Pad_1.0x1.0mm, symbol Connector:TestPoint
- added TP10: TestPoint, TestPoint:TestPoint_Pad_D3.0mm, symbol Connector:TestPoint
- added U1: MAX17048G_T10, MAX17048G_T10:SON50P200X200X80-9N, symbol MAX17048G_T10:MAX17048G_T10
- L1: footprint Inductor_SMD:L_6.3x6.3_H3 -> Inductor_SMD:L_1008_2520Metric
- L3: footprint Inductor_SMD:L_6.3x6.3_H3 -> IHLP2020ABER1R0M01:IND_R2M01_VIS
- R14: value R -> 430
- S3, S4: footprint PTS815SJM250SMTRLFS -> SamacSys:PTS815SJM250SMTRLFS
- TH1: value Thermistor -> B25/85 3435K; footprint Resistor_SMD:R_0402_1005Metric -> Resistor_SMD:R_0805_2012Metric
Connections:
- net +3.3V: now also J6.1 (Pin_1), JP1.1 (A), TP5.1
- net +5V_CHARGE: now also R14.1, C32.2, TP1.1; no longer D1.2 (A)
- net +5V_OUT: now also R15.1, J7.01 (VCC), J9.2 (Pin_2), TP2.1; no longer D2.2 (A)
- net +BATT: now also TP3.1, U1.2 (CELL), U1.3 (VDD)
- net 5VEN: now also C33.1, JP1.2 (B), R29.1, TP7.1
- net GND: now also D1.1 (K), D2.1 (K), R1.1, R2.1, C31.2, C32.1, C33.2, J2.5 (Pin_5), J5.5 (Pin_5), J7.04 (GND), J7.SH1 (SHIELD), J7.SH2 (SHIELD), J8.MP1, J8.MP2, J8.MP3, J8.MP4, J9.1 (Pin_1), R26.2, R27.2, R28.1, R29.2, TP10.1, U1.1 (CTG), U1.4 (GND), U1.6 (QSTRT), U1.9 (EP); no longer R1.2, R14.2, R15.2, R2.2
- net INT_BQ: now also U5.13 (PA3)
- net INT_MAX: now also U5.14 (PA4), U1.5 (~{ALERT})
- net LED: now also D5.1 (K)
- net REACT: now also J2.3 (Pin_3), R27.1, TP8.1
- net RX: now also J2.2 (Pin_2)
- net SCL: now also U1.7 (SCL)
- net SDA: now also U1.8 (SDA)
- net SWCLK: now also J5.3 (Pin_3)
- net SWDIO: now also J5.4 (Pin_4)
- net SWO: now also J5.2 (Pin_2)
- net TRIG: now also J2.4 (Pin_4), R28.2, TP9.1
- net TX: now also J2.1 (Pin_1)
- net VDD: now also J5.1 (Pin_1), J8.3
- net V_SYS: now also C31.1, J8.1, TP4.1
- net O/X: now reaches R10.1, R7.1, S3.3 (NO1), S3.4 (NO2)
- net O/X: now also J6.2 (Pin_2)
- net at J4.B5 (CC2): now also R2.2; no longer R2.1
- net at J4.A5 (CC1): now also R1.2; no longer R1.1
- net EN3V3 renamed VIN_STM
- net VIN_STM: now also J8.2, TP6.1
- net OFF renamed ON/OFF
- new net: D5.2 (A), R26.1
- new net: D1.2 (A), R14.2
- new net: D2.2 (A), R15.2
- no-connect marks 4 -> 27
Other:
- note added: "+5V: USB A, pin connector"
- note added: "- czy gpio REACT/TRIG potrzebuje pull-up pull-down? Masz internall pullup/pulldown, może to wystarczy - czy UART TX/RX potrezbuje pull-up pull-down? - DISP_IRQ/INT_MAX/INT_BQ wtf???"
- note added: "BQ24296"
- note added: "Mounting Holes / Fiducials"
- note added: "O/X BTN"
- note added: "OK - Mounting holes - Dodaj MAX / BQ ISR piny do MCU - USB A receptacle - 5VEN, REACT, TRIG pulldown? ZROB - Test pointy - GND pours / stiching vias?"
- note added: "SINK - consumes power / wall adapter -> power supply SOURCE - provides power / power supply -> circuit load"
- note added: "Test Points"
- note added: "Toggle MCU power"
- note added: "USB-C Sink 5V@3A (CC pull-down)"
- note added: "USB-C Source 5V@3A (CC pull-up)"
- note removed: "- czy gpio REACT/TRIG potrzebuje pull-up pull-down? - czy UART TX/RX potrezbuje pull-up pull-down? - DISP_IRQ/INT_MAX/INT_BQ wtf???"
- note removed: "BQ24296 / Efuse"
- note removed: "Toggle MCU power src (!!!!!!!!! WTF??) Chyba symbol/footprint jest nie ok"
- note removed: "USB-C Sink 5V@3A"
- note removed: "USB-C Source 5V@3A"
- moved on the sheet: BT1, BT2, C1, C10, C11, C12, C13, C14, C2, C22, C23, C3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
